File: power.sch (EAGLE design)
At the start: 19 parts, among them IC1 BLUETOOTH-RN42 HID, Q1 MOSFET-NCHANNELSMD, Q2 MOSFET-NCHANNELSMD, U1 MCP73831, X1 Micro USB

Commit message: Starting to flesh this out
Parts:
- removed IC1: BLUETOOTH-RN42 HID, SparkFun-RF:BLUETOOTH-RN41"
- removed JP8: (no value), SparkFun:M02PTH
- removed R2, R5: 10K, SparkFun:RESISTOR0603-RES
Connections:
- removed net CTS: R2.1
- removed net CTS_5V: R2.2
- removed net N$1: IC1.UARTRX
- removed net N$10: IC1.PIO5
- removed net N$11: IC1.VDD
- removed net N$2: IC1.UARTTX
- removed net N$3: IC1.UARTRTS
- removed net N$4: IC1.UARTCTS
- removed net N$5: IC1.USBD-
- removed net N$6: IC1.USBD+
- removed net N$8: IC1.PIO2
- removed net N$9: IC1.PIO4
- removed net RX: R5.1
- removed net RX_5V: R5.2
- net GND: no longer IC1.GND, IC1.GND1, IC1.GND2, IC1.GND3, JP8.1
- net VCC: no longer JP8.2
Other:
- moved on the sheet: Q1, Q2, R1, R3, R4, R7, R8

Commit message: Updating with changes
Parts:
- removed C3, C4: 4.7uF, SparkFun:CAP0402-CAP
- removed Q1, Q2: MOSFET-NCHANNELSMD, SparkFun:MOSFET-NCHANNELSMD
- removed R3, R4, R7, R8: 10K, SparkFun:RESISTOR0603-RES
- removed R6: 330, SparkFun:RESISTOR0402-RES
- removed R9: 2K, SparkFun:RESISTOR0402-RES
- added C1, C2: 4.7uF, SparkFun-Capacitors:1.0UF-25V-+80/-20(0805)"
- added R2: 2k, SparkFun-Resistors:0.22OHM-1/4W-1%(0805)
- R1: value 10k -> 330
Connections:
- removed net 3.3V: Q1.G, Q2.G, R3.1, R7.1
- removed net RTS: Q2.S, R7.2
- removed net RTS_5V: Q2.D, R8.2
- removed net TX: Q1.S, R3.2
- removed net TX_5V: Q1.D, R4.2
- net GND: now also C1.2, C2.2, R2.1; no longer C3.2, C4.2, R9.2
- net N$12: now also R1.2; no longer R6.1
- net PROG: now also R2.2; no longer R9.1
- net VCC: now also C2.1; no longer C4.1, R4.1, R8.1
- net VIN: now also C1.1, R1.1; no longer C3.1, R6.2
Other:
- moved on the sheet: R1

Commit message: More updates
Parts:
- added IC1: CAT4101, User-Submitted:CAT4101
- added JP1: RA 6Pin SMD, SparkFun-Connectors:M06SMD
- added U2: Tiny85-20-SMT, SparkFun-DigitalIC:ATTINY45TINY85-20-SMT
Connections:
- removed net VCC: C2.1, JP7.2, U1.VBAT
- new net VBAT: C2.1, JP1.6, JP7.2, U1.VBAT
- net GND: now also JP1.1
Other:
- note removed: "0.1""
- note removed: "Connection to 3.7V System"
Changed lines of the file:
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@@
 <layer number="56" name="wert" color="7" fill="1" visible="no" active="no"/>
 <layer number="57" name="tCAD" color="7" fill="1" visible="no" active="no"/>
+<layer number="59" name="tCarbon" color="7" fill="1" visible="no" active="no"/>
+<layer number="60" name="bCarbon" color="7" fill="1" visible="no" active="no"/>
 <layer number="90" name="Modules" color="5" fill="1" visible="yes" active="yes"/>
 <layer number="91" name="Nets" color="2" fill="1" visible="yes" active="yes"/>
@@
 <layer number="112" name="tSilk" color="7" fill="1" visible="yes" active="yes"/>
 <layer number="113" name="IDFDebug" color="4" fill="1" visible="yes" active="yes"/>
+<layer number="114" name="Badge_Outline" color="7" fill="1" visible="yes" active="yes"/>
+<layer number="115" name="ReferenceISLANDS" color="7" fill="1" visible="yes" active="yes"/>
 <layer number="116" name="Patch_BOT" color="9" fill="4" visible="yes" active="yes"/>
+<layer number="118" name="Rect_Pads" color="7" fill="1" visible="yes" active="yes"/>
 <layer number="121" name="_tsilk" color="7" fill="1" visible="yes" active="yes"/>
 <layer number="122" name="_bsilk" color="7" fill="1" visible="yes" active="yes"/>
@@
 <layer number="127" name="_tValues" color="7" fill="1" visible="yes" active="yes"/>
 <layer number="128" name="_bValues" color="7" fill="1" visible="yes" active="yes"/>
+<layer number="129" name="Mask" color="7" fill="1" visible="yes" active="yes"/>
 <layer number="131" name="tAdjust" color="7" fill="1" visible="yes" active="yes"/>
 <layer number="132" name="bAdjust" color="7" fill="1" visible="yes" active="yes"/>
@@
 <layer number="251" name="SMDround" color="12" fill="11" visible="no" active="no"/>
 <layer number="254" name="cooling" color="7" fill="1" visible="yes" active="yes"/>
+<layer number="255" name="routoute" color="7" fill="1" visible="yes" active="yes"/>
 </layers>
 <schematic xreflabel="%F%N/%S.%C%R" xrefpart="/%S.%C%R">
@@
 <part name="GND15" library="SparkFun" deviceset="GND" device=""/>
 <part name="GND14" library="SparkFun" deviceset="GND" device=""/>
-<part name="GND17" library="SparkFun" deviceset="GND" device=""/>
+<part name="CLONE" library="SparkFun" deviceset="GND" device=""/>
 <part name="GND18" library="SparkFun" deviceset="GND" device=""/>
 <part name="U1" library="SparkFun" deviceset="MCP73831" device=""/>
@@
 <part name="C1" library="SparkFun-Capacitors" deviceset="1.0UF-25V-+80/-20(0805)" device="&quot;" value="4.7uF"/>
 <part name="C2" library="SparkFun-Capacitors" deviceset="1.0UF-25V-+80/-20(0805)" device="&quot;" value="4.7uF"/>
+<part name="JP1" library="SparkFun-Connectors" deviceset="M06" device="SMD" value="RA 6Pin SMD"/>
+<part name="U2" library="SparkFun-DigitalIC" deviceset="ATTINY45" device="TINY85-20-SMT" value="Tiny85-20-SMT"/>
+<part name="GND2" library="SparkFun" deviceset="GND" device=""/>
+<part name="IC1" library="User-Submitted" deviceset="CAT4101" device=""/>
 </parts>
 <sheets>
 <sheet>
 <plain>
-<wire x1="236.22" y1="152.4" x2="254" y2="152.4" width="0.2032" layer="97" style="longdash"/>
-<wire x1="254" y1="152.4" x2="254" y2="124.46" width="0.2032" layer="97" style="longdash"/>
-<wire x1="254" y1="124.46" x2="236.22" y2="124.46" width="0.2032" layer="97" style="longdash"/>
-<wire x1="236.22" y1="124.46" x2="236.22" y2="152.4" width="0.2032" layer="97" style="longdash"/>
 <text x="167.64" y="142.24" size="1.778" layer="97">Set for 500mA charging</text>
-<text x="228.346" y="154.432" size="1.778" layer="97">Connection to 3.7V System</text>
-<text x="243.586" y="148.59" size="1.778" layer="97">0.1"</text>
 <text x="134.874" y="144.272" size="1.778" layer="97">microUSB</text>
 </plain>
@@
 <instance part="GND15" gate="1" x="147.32" y="127"/>
 <instance part="GND14" gate="1" x="210.82" y="119.38"/>
-<instance part="GND17" gate="1" x="154.94" y="119.38"/>
+<instance part="CLONE" gate="1" x="154.94" y="119.38"/>
 <instance part="GND18" gate="1" x="193.04" y="124.46"/>
 <instance part="U1" gate="G$1" x="182.88" y="132.08"/>
@@
 <instance part="C1" gate="G$1" x="154.94" y="127"/>
 <instance part="C2" gate="G$1" x="210.82" y="127"/>
+<instance part="JP1" gate="G$1" x="205.74" y="91.44"/>
+<instance part="U2" gate="G$1" x="172.72" y="78.74"/>
+<instance part="GND2" gate="1" x="213.36" y="81.28"/>
+<instance part="IC1" gate="G$1" x="205.74" y="50.8"/>
 </instances>
 <busses>
 </busses>
 <nets>
-<net name="VCC" class="0">
+<net name="VBAT" class="0">
 <segment>
 <wire x1="210.82" y1="132.08" x2="210.82" y2="134.62" width="0.1524" layer="91"/>
 <wire x1="193.04" y1="134.62" x2="210.82" y2="134.62" width="0.1524" layer="91"/>
 <wire x1="210.82" y1="134.62" x2="220.98" y2="134.62" width="0.1524" layer="91"/>
-<wire x1="220.98" y1="134.62" x2="243.84" y2="134.62" width="0.1524" layer="91"/>
+<wire x1="220.98" y1="134.62" x2="231.14" y2="134.62" width="0.1524" layer="91"/>
 <wire x1="220.98" y1="137.16" x2="220.98" y2="134.62" width="0.1524" layer="91"/>
 <junction x="210.82" y="134.62"/>
 <junction x="220.98" y="134.62"/>
-<label x="198.12" y="134.62" size="1.778" layer="95"/>
+<label x="231.14" y="134.62" size="1.778" layer="95"/>
 <pinref part="U1" gate="G$1" pin="VBAT"/>
 <pinref part="JP7" gate="G$1" pin="2"/>
 <pinref part="C2" gate="G$1" pin="1"/>
 </segment>
+<segment>
+<pinref part="JP1" gate="G$1" pin="6"/>
+<wire x1="210.82" y1="99.06" x2="213.36" y2="99.06" width="0.1524" layer="91"/>
+<label x="213.36" y="99.06" size="1.778" layer="95"/>
+</segment>
 </net>
 <net name="GND" class="0">
@@
 <segment>
 <wire x1="154.94" y1="121.92" x2="154.94" y2="124.46" width="0.1524" layer="91"/>
-<pinref part="GND17" gate="1" pin="GND"/>
+<pinref part="CLONE" gate="1" pin="GND"/>
 <pinref part="C1" gate="G$1" pin="2"/>
 </segment>
@@
 <pinref part="GND1" gate="1" pin="GND"/>
 </segment>
+<segment>
+<pinref part="JP1" gate="G$1" pin="1"/>
+<wire x1="210.82" y1="86.36" x2="213.36" y2="86.36" width="0.1524" layer="91"/>
+<pinref part="GND2" gate="1" pin="GND"/>
+<wire x1="213.36" y1="86.36" x2="213.36" y2="83.82" width="0.1524" layer="91"/>
+</segment>
 </net>
