File: power.sch (EAGLE design)
At the start: 11 parts, among them IC1 UC27775, U1 MCP73831, U2 Tiny85-20-SMT, X1 Micro USB

Commit message: Putting more info on this thing to help me out
Parts:
- added J2: USB-MINIB-TH-VERTICAL-5PIN, mine:USB-MINIB-TH-VERTICAL-5PIN
Connections:
- new net N$2: J2.D-, JP1.4
- new net N$3: J2.D+, JP1.3
- new net VCC: IC1.SWITCH, J2.VBUS, JP1.5
- net GND: now also IC1.GND, J2.GND
- net VBAT: now also IC1.VIN
Other:
- moved on the sheet: IC1, JP1, U2
Changed lines of the file:
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@@
 <part name="JP1" library="mine" deviceset="M06" device="SMD-NOHOLES" value="RA 6Pin SMD"/>
 <part name="IC1" library="mine" deviceset="UC27775" device=""/>
+<part name="GND3" library="SparkFun" deviceset="GND" device=""/>
+<part name="J2" library="mine" deviceset="USB-MINIB-TH-VERTICAL" device="-5PIN"/>
 </parts>
 <sheets>
@@
 <instance part="C1" gate="G$1" x="154.94" y="127"/>
 <instance part="C2" gate="G$1" x="210.82" y="127"/>
-<instance part="U2" gate="G$1" x="172.72" y="78.74"/>
-<instance part="GND2" gate="1" x="213.36" y="81.28"/>
-<instance part="JP1" gate="G$1" x="205.74" y="91.44"/>
-<instance part="IC1" gate="G$1" x="205.74" y="55.88"/>
+<instance part="U2" gate="G$1" x="165.1" y="45.72"/>
+<instance part="GND2" gate="1" x="177.8" y="73.66"/>
+<instance part="JP1" gate="G$1" x="170.18" y="83.82"/>
+<instance part="IC1" gate="G$1" x="208.28" y="48.26"/>
+<instance part="GND3" gate="1" x="190.5" y="73.66"/>
+<instance part="J2" gate="G$1" x="195.58" y="78.74"/>
 </instances>
 <busses>
@@
 </segment>
 <segment>
-<wire x1="210.82" y1="99.06" x2="213.36" y2="99.06" width="0.1524" layer="91"/>
-<label x="213.36" y="99.06" size="1.778" layer="95"/>
+<wire x1="175.26" y1="91.44" x2="177.8" y2="91.44" width="0.1524" layer="91"/>
+<label x="177.8" y="91.44" size="1.778" layer="95"/>
 <pinref part="JP1" gate="G$1" pin="6"/>
+</segment>
+<segment>
+<pinref part="IC1" gate="G$1" pin="VIN"/>
+<wire x1="198.12" y1="53.34" x2="195.58" y2="53.34" width="0.1524" layer="91"/>
+<label x="190.5" y="53.34" size="1.778" layer="95"/>
 </segment>
 </net>
@@
 </segment>
 <segment>
-<wire x1="210.82" y1="86.36" x2="213.36" y2="86.36" width="0.1524" layer="91"/>
+<wire x1="175.26" y1="78.74" x2="177.8" y2="78.74" width="0.1524" layer="91"/>
 <pinref part="GND2" gate="1" pin="GND"/>
-<wire x1="213.36" y1="86.36" x2="213.36" y2="83.82" width="0.1524" layer="91"/>
+<wire x1="177.8" y1="78.74" x2="177.8" y2="76.2" width="0.1524" layer="91"/>
 <pinref part="JP1" gate="G$1" pin="1"/>
+</segment>
+<segment>
+<pinref part="IC1" gate="G$1" pin="GND"/>
+<wire x1="198.12" y1="40.64" x2="195.58" y2="40.64" width="0.1524" layer="91"/>
+<label x="190.5" y="40.64" size="1.778" layer="95"/>
+</segment>
+<segment>
+<wire x1="193.04" y1="78.74" x2="190.5" y2="78.74" width="0.1524" layer="91"/>
+<wire x1="190.5" y1="78.74" x2="190.5" y2="76.2" width="0.1524" layer="91"/>
+<pinref part="GND3" gate="1" pin="GND"/>
+<pinref part="J2" gate="G$1" pin="GND"/>
 </segment>
 </net>
@@
 </segment>
 </net>
+<net name="N$2" class="0">
+<segment>
+<pinref part="JP1" gate="G$1" pin="4"/>
+<wire x1="175.26" y1="86.36" x2="193.04" y2="86.36" width="0.1524" layer="91"/>
+<pinref part="J2" gate="G$1" pin="D-"/>
+</segment>
+</net>
+<net name="N$3" class="0">
+<segment>
+<pinref part="JP1" gate="G$1" pin="3"/>
+<wire x1="175.26" y1="83.82" x2="193.04" y2="83.82" width="0.1524" layer="91"/>
+<pinref part="J2" gate="G$1" pin="D+"/>
+</segment>
+</net>
+<net name="VCC" class="0">
+<segment>
+<pinref part="IC1" gate="G$1" pin="SWITCH"/>
+<wire x1="198.12" y1="50.8" x2="195.58" y2="50.8" width="0.1524" layer="91"/>
+<label x="190.5" y="50.8" size="1.778" layer="95"/>
+</segment>
+<segment>
+<wire x1="193.04" y1="88.9" x2="190.5" y2="88.9" width="0.1524" layer="91"/>
+<label x="185.42" y="88.9" size="1.778" layer="95"/>
+<pinref part="J2" gate="G$1" pin="VBUS"/>
+</segment>
+<segment>
+<pinref part="JP1" gate="G$1" pin="5"/>
+<wire x1="175.26" y1="88.9" x2="177.8" y2="88.9" width="0.1524" layer="91"/>
+<label x="177.8" y="88.9" size="1.778" layer="95"/>
+</segment>
+</net>
