File: power.brd (EAGLE design)
At the start: 27.6 x 17.8 mm, 11 parts, among them IC1 UC27775, U1 MCP73831, U2 Tiny85-20-SMT, X1 Micro USB

Commit message: Putting more info on this thing to help me out
Parts:
- added J2: USB-MINIB-TH-VERTICAL-5PIN, mine:USB-MINIB-TH-VERTICAL
Connections:
- new net N$2: J2.D-, JP1.4
- new net N$3: J2.D+, JP1.3
- new net VCC: IC1.4, J2.VBUS, JP1.5
- net GND: now also J2.GND
- net VBAT: now also IC1.5
Other:
- board text added: "1000mAh LiPo"
- board text added: "400mAh LiPo"
- board text added: "850mAh LiPo"
- board text added: "RN42-HID Module"
Changed lines of the file:
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@@
 <drawing>
 <settings>
-<setting alwaysvectorfont="no"/>
+<setting alwaysvectorfont="yes"/>
 <setting verticaltext="up"/>
 </settings>
-<grid distance="0.025" unitdist="inch" unit="inch" style="lines" multiple="1" display="no" altdistance="0.025" altunitdist="inch" altunit="inch"/>
+<grid distance="0.0125" unitdist="inch" unit="inch" style="lines" multiple="1" display="no" altdistance="0.025" altunitdist="inch" altunit="inch"/>
 <layers>
 <layer number="1" name="Top" color="4" fill="1" visible="yes" active="yes"/>
@@
 <layer number="50" name="dxf" color="7" fill="1" visible="no" active="no"/>
 <layer number="51" name="tDocu" color="7" fill="1" visible="yes" active="yes"/>
-<layer number="52" name="bDocu" color="7" fill="1" visible="yes" active="yes"/>
+<layer number="52" name="bDocu" color="23" fill="1" visible="yes" active="yes"/>
 <layer number="53" name="tGND_GNDA" color="7" fill="9" visible="no" active="no"/>
 <layer number="54" name="bGND_GNDA" color="1" fill="9" visible="no" active="no"/>
@@
 <wire x1="27.61" y1="17.77" x2="0" y2="17.77" width="0" layer="20"/>
 <wire x1="0" y1="17.77" x2="0" y2="0" width="0" layer="20"/>
-<circle x="14.605" y="3.81" radius="0.635" width="0.4064" layer="1"/>
-<circle x="12.7" y="3.81" radius="0.635" width="0.4064" layer="1"/>
-<circle x="10.795" y="3.81" radius="0.635" width="0.4064" layer="1"/>
-<circle x="16.51" y="3.81" radius="0.635" width="0.4064" layer="1"/>
-<circle x="19.685" y="3.81" radius="1.419903125" width="0.4064" layer="1"/>
-<circle x="7.62" y="3.81" radius="1.419903125" width="0.4064" layer="1"/>
+<text x="8.89" y="23.495" size="1.778" layer="51">400mAh LiPo</text>
+<rectangle x1="29.845" y1="0" x2="59.055" y2="17.78" layer="52"/>
+<text x="50.165" y="9.8425" size="1.016" layer="51" rot="R180">RN42-HID Module</text>
+<dimension x1="50.8" y1="0" x2="50.8" y2="33.5" x3="52.07" y3="16.75" textsize="1.016" layer="51"/>
+<dimension x1="0" y1="37.465" x2="50.8" y2="37.465" x3="25.4" y3="35.56" textsize="1.016" layer="51"/>
+<text x="8.89" y="33.02" size="1.778" layer="51">1000mAh LiPo</text>
+<dimension x1="0" y1="29.45" x2="48.27" y2="29.45" x3="24.135" y3="31.114996875" textsize="1.016" layer="51"/>
+<text x="9.525" y="28.575" size="1.778" layer="51">850mAh LiPo</text>
+<dimension x1="51.435" y1="-0.05" x2="51.435" y2="29.45" x3="50.165" y3="14.7" textsize="1.016" layer="51"/>
+<dimension x1="35" y1="0" x2="34.925" y2="24.765" x3="36.242096875" y3="12.386375" textsize="1.016" layer="51"/>
+<dimension x1="0" y1="25" x2="35" y2="25" x3="17.5" y3="26.035" textsize="1.016" layer="51"/>
 </plain>
 <attributes>
@@
 <attribute name="PROD_ID" value="IC-09092" x="18.415" y="11.43" size="1.778" layer="28" rot="MR0" display="off"/>
 </element>
-<element name="JP1" library="mine" package="1X06-SMD-NOHOLES" value="RA 6Pin SMD" x="28.575" y="8.89" rot="MR270">
+<element name="JP1" library="mine" package="1X06-SMD-NOHOLES" value="RA 6Pin SMD" x="28.575" y="8.89" smashed="yes" rot="MR270">
 <attribute name="PROD_ID" value="CONN-08971" x="28.575" y="8.89" size="1.778" layer="28" rot="MR270" display="off"/>
+<attribute name="NAME" x="26.67" y="10.795" size="0.8128" layer="26" rot="MR270"/>
 </element>
 <element name="IC1" library="mine" package="TO263_5" value="UC27775" x="14.605" y="11.43" rot="R90">
 <attribute name="MF" value="TI" x="14.605" y="11.43" size="1.778" layer="27" rot="R90" display="off"/>
+</element>
+<element name="J2" library="mine" package="USB-MINIB-TH-VERTICAL" value="USB-MINIB-TH-VERTICAL-5PIN" x="12.7" y="2.54">
+<attribute name="PROD_ID" value="CONN-08193" x="12.7" y="2.54" size="1.016" layer="27" display="off"/>
 </element>
 </elements>
@@
 <contactref element="C2" pad="1"/>
 <contactref element="JP1" pad="6"/>
+<contactref element="IC1" pad="5"/>
+<wire x1="23.575" y1="2.54" x2="22.605" y2="14.83" width="0" layer="19" extent="1-16"/>
+<wire x1="7.73" y1="12.43" x2="22.605" y2="14.83" width="0" layer="19" extent="1-16"/>
 <wire x1="3.44" y1="14.605" x2="7.73" y2="12.43" width="0" layer="19" extent="16-16"/>
 <wire x1="1.8749" y1="9.205" x2="3.44" y2="14.605" width="0" layer="19" extent="16-16"/>
-<wire x1="23.575" y1="2.54" x2="7.73" y2="12.43" width="0" layer="19" extent="1-16"/>
 </signal>
 <signal name="VIN">
@@
 <contactref element="C1" pad="2"/>
 <contactref element="C2" pad="2"/>
+<contactref element="JP1" pad="1"/>
 <contactref element="IC1" pad="3"/>
-<contactref element="JP1" pad="1"/>
+<contactref element="J2" pad="GND"/>
+<wire x1="22.605" y1="11.43" x2="23.575" y2="15.24" width="0" layer="19" extent="1-16"/>
+<wire x1="7.73" y1="10.43" x2="22.605" y2="11.43" width="0" layer="19" extent="1-16"/>
 <wire x1="1.8749" y1="8.255" x2="7.73" y2="10.43" width="0" layer="19" extent="16-16"/>
 <wire x1="1.64" y1="4.445" x2="1.8749" y2="8.255" width="0" layer="19" extent="16-16"/>
 <wire x1="1.64" y1="1.905" x2="1.64" y2="4.445" width="0" layer="19" extent="16-16"/>
 <wire x1="4.555" y1="4.415" x2="1.64" y2="4.445" width="0" layer="19" extent="1-16"/>
-<wire x1="23.575" y1="15.24" x2="1.64" y2="1.905" width="0" layer="19" extent="1-16"/>
+<wire x1="15.875" y1="2.54" x2="1.64" y2="1.905" width="0" layer="19" extent="16-16"/>
 <wire x1="1.64" y1="14.605" x2="1.8749" y2="8.255" width="0" layer="19" extent="16-16"/>
-<wire x1="22.605" y1="11.43" x2="23.575" y2="15.24" width="0" layer="19" extent="1-1"/>
 </signal>
 <signal name="N$12">
@@
 <wire x1="1.8749" y1="7.305" x2="1.79" y2="12.065" width="0" layer="19" extent="1-16"/>
 </signal>
+<signal name="N$2">
+<contactref element="JP1" pad="4"/>
+<contactref element="J2" pad="D-"/>
+<wire x1="11.1125" y1="2.54" x2="23.575" y2="7.62" width="0" layer="19" extent="16-16"/>
+</signal>
+<signal name="N$3">
+<contactref element="JP1" pad="3"/>
+<contactref element="J2" pad="D+"/>
+<wire x1="12.7" y1="2.54" x2="23.575" y2="10.16" width="0" layer="19" extent="16-16"/>
+</signal>
+<signal name="VCC">
+<contactref element="IC1" pad="4"/>
+<contactref element="JP1" pad="5"/>
+<contactref element="J2" pad="VBUS"/>
+<wire x1="23.575" y1="5.08" x2="22.605" y2="13.13" width="0" layer="19" extent="1-16"/>
+<wire x1="9.525" y1="2.54" x2="23.575" y2="5.08" width="0" layer="19" extent="16-16"/>
+</signal>
 </signals>
